File: CESP.kicad_pcb (KiCad board)
At the start: 2 copper layers, 55.9 x 44.7 mm, 9 parts

Commit message: Added some BS
Parts:
- removed the LED-1206 at (201.5, 99.9)
- removed SOIC24: VAL**, SOIC24
- removed the TSSOP14 at (199.1, 134.7)
- added U***: 20TEX-ELL300, 20TEX-ELL300, F.Cu at (190.1, 117.2)
