File: CESP.sch (KiCad schematic (older format))
At the start: 5 parts

Commit message: Added some BS
Parts:
- added IC? (x2): AT89S2051-S, SO20, symbol AT89S2051-S
Changed lines of the file:
@@
-EESchema Schematic File Version 2  date 1/24/2014 12:04:40 AM
+EESchema Schematic File Version 2
 LIBS:power
 LIBS:device
@@
 Sheet 1 1
 Title ""
-Date "24 jan 2014"
+Date "6 feb 2014"
 Rev ""
 Comp ""
@@
 Text Notes 4450 4650 0    80   ~ 0
 NOTE: THIS IS JUST A TEST BOARD\nREMOVE ALL COMPONENTS AND CREATE YOUR OWN\nINCLUDE SCHEMATIC HOOKUPS/NETLIST
+$Comp
+L AT89S2051-S IC?
+U 1 1 52F3B2C9
+P 2800 1400
+F 0 "IC?" H 1850 2400 40  0000 C CNN
+F 1 "AT89S2051-S" H 3550 500 40  0000 C CNN
+F 2 "SO20" H 2800 1400 30  0000 C CIN
+F 3 "" H 2800 1400 60  0000 C CNN
+	1    2800 1400
+	1    0    0    -1
+$EndComp
+$Comp
+L AT89S2051-S IC?
+U 1 1 52F3B2D8
+P 3650 6350
+F 0 "IC?" H 2700 7350 40  0000 C CNN
+F 1 "AT89S2051-S" H 4400 5450 40  0000 C CNN
+F 2 "SO20" H 3650 6350 30  0000 C CIN
+F 3 "" H 3650 6350 60  0000 C CNN
+	1    3650 6350
+	1    0    0    -1
+$EndComp
 $EndSCHEMATC
